File: curve_tracer/curve_tracer.kicad_sch (KiCad schematic)
At the start: 6 parts, among them J1 Conn_01x10, J2 Conn_01x03, J3 Conn_01x30, U1 LM358

Commit message: fix an issue
Parts:
- added D1: LED, symbol Device:LED
Connections:
- net GND: now also D1.1 (K)
- net +5V: now reaches J3.16 (Pin_16)
- net +5V: now also J1.1 (Pin_1), U1.8 (V+), D1.2 (A)
- removed net +3V3: J1.1 (Pin_1), J3.1 (Pin_1), U1.8 (V+)
